Commit message: ATT

File: install/sobot_drive/share/sobot_drive/ros2_control/diffbot.ros2_control.xacro (robot description, xacro)
@@ -1 +1,33 @@
-/dev_ws/src/sobot_drive/description/ros2_control/diffbot.ros2_control.xacro
+<?xml version="1.0"?>
+<robot xmlns:xacro="http://www.ros.org/wiki/xacro">
+  <xacro:macro name="diffbot_ros2_control" params="name prefix use_mock_hardware">
+    <ros2_control name="${name}" type="system">
+      <xacro:unless value="${use_mock_hardware}">
+        <hardware>
+          <plugin>sobot_drive/SobotDriveHardware</plugin>
+          <param name="example_param_hw_start_duration_sec">0</param>
+          <param name="example_param_hw_stop_duration_sec">3.0</param>
+          <param name="device">/dev/ttyACM0</param>
+          <param name="baud_rate">57600</param>
+          <param name="timeout_ms">1000</param>
+        </hardware>
+      </xacro:unless>
+      <xacro:if value="${use_mock_hardware}">
+        <hardware>
+          <plugin>mock_components/GenericSystem</plugin>
+          <param name="calculate_dynamics">true</param>
+        </hardware>
+      </xacro:if>
+      <joint name="${prefix}left_wheel_joint">
+        <command_interface name="velocity"/>
+        <state_interface name="position"/>
+        <state_interface name="velocity"/>
+      </joint>
+      <joint name="${prefix}right_wheel_joint">
+        <command_interface name="velocity"/>
+        <state_interface name="position"/>
+        <state_interface name="velocity"/>
+      </joint>
+    </ros2_control>
+  </xacro:macro>
+</robot>

File: install/sobot_drive/share/sobot_drive/urdf/diffbot.urdf.xacro (robot description, xacro)
@@ -1 +1,10 @@
-/dev_ws/src/sobot_drive/description/urdf/diffbot.urdf.xacro
+<?xml version="1.0"?>
+<!-- Basic differential drive mobile base -->
+<robot xmlns:xacro="http://www.ros.org/wiki/xacro" name="diffdrive_robot">
+  <xacro:arg name="prefix" default="" />
+  <xacro:include filename="robot_core.xacro" />
+  <!-- Import diffbot ros2_control description -->
+  <xacro:include filename="$(find sobot_drive)/ros2_control/diffbot.ros2_control.xacro" />
+  <xacro:diffbot_ros2_control
+    name="DiffBot" prefix="$(arg prefix)" use_mock_hardware="$(arg use_mock_hardware)"/>
+</robot>

Commit message: ATT

File: install/sobot_drive/share/sobot_drive/ros2_control/diffbot.ros2_control.xacro (robot description, xacro)
@@ -1,33 +1 @@
-<?xml version="1.0"?>
-<robot xmlns:xacro="http://www.ros.org/wiki/xacro">
-  <xacro:macro name="diffbot_ros2_control" params="name prefix use_mock_hardware">
-    <ros2_control name="${name}" type="system">
-      <xacro:unless value="${use_mock_hardware}">
-        <hardware>
-          <plugin>sobot_drive/SobotDriveHardware</plugin>
-          <param name="example_param_hw_start_duration_sec">0</param>
-          <param name="example_param_hw_stop_duration_sec">3.0</param>
-          <param name="device">/dev/ttyACM0</param>
-          <param name="baud_rate">57600</param>
-          <param name="timeout_ms">1000</param>
-        </hardware>
-      </xacro:unless>
-      <xacro:if value="${use_mock_hardware}">
-        <hardware>
-          <plugin>mock_components/GenericSystem</plugin>
-          <param name="calculate_dynamics">true</param>
-        </hardware>
-      </xacro:if>
-      <joint name="${prefix}left_wheel_joint">
-        <command_interface name="velocity"/>
-        <state_interface name="position"/>
-        <state_interface name="velocity"/>
-      </joint>
-      <joint name="${prefix}right_wheel_joint">
-        <command_interface name="velocity"/>
-        <state_interface name="position"/>
-        <state_interface name="velocity"/>
-      </joint>
-    </ros2_control>
-  </xacro:macro>
-</robot>
+/home/rods/dev_ws/src/sobot_drive/description/ros2_control/diffbot.ros2_control.xacro

File: install/sobot_drive/share/sobot_drive/urdf/diffbot.urdf.xacro (robot description, xacro)
@@ -1,10 +1 @@
-<?xml version="1.0"?>
-<!-- Basic differential drive mobile base -->
-<robot xmlns:xacro="http://www.ros.org/wiki/xacro" name="diffdrive_robot">
-  <xacro:arg name="prefix" default="" />
-  <xacro:include filename="robot_core.xacro" />
-  <!-- Import diffbot ros2_control description -->
-  <xacro:include filename="$(find sobot_drive)/ros2_control/diffbot.ros2_control.xacro" />
-  <xacro:diffbot_ros2_control
-    name="DiffBot" prefix="$(arg prefix)" use_mock_hardware="$(arg use_mock_hardware)"/>
-</robot>
+/home/rods/dev_ws/src/sobot_drive/description/urdf/diffbot.urdf.xacro

File: src/sobot_drive/description/urdf/diffbot.urdf.xacro (robot description, xacro)
@@ -3,4 +3,5 @@
 <robot xmlns:xacro="http://www.ros.org/wiki/xacro" name="diffdrive_robot">
   <xacro:arg name="prefix" default="" />
+  <xacro:arg name="use_mock_hardware" default="false" />
   <xacro:include filename="robot_core.xacro" />
   <!-- Import diffbot ros2_control description -->

File: src/sobot_drive/description/urdf/robot_core.xacro (robot description, xacro)
@@ -32,5 +32,5 @@
         <visual>
             <geometry>
-                <mesh filename="package://sobot/description/meshes/sobot_chassis.dae" scale="1 1 1"/>
+                <mesh filename="package://sobot_drive/meshes/sobot_chassis.dae" scale="1 1 1"/>
             </geometry>
             <material name="grey"/>
@@ -60,5 +60,5 @@
                 <origin xyz="0.0 0.0 0.0" rpy="-1.57 0 0" />
             <geometry>
-                <mesh filename="package://sobot/description/meshes/sobot_wheel.dae" scale="1 1 1"/> <!-- Colocar o arquivo STL-->
+                <mesh filename="package://sobot_drive/meshes/sobot_wheel.dae" scale="1 1 1"/> <!-- Colocar o arquivo STL-->
             </geometry>
         </visual>
@@ -86,5 +86,5 @@
             <origin xyz="0 0 0" rpy="1.57 0 0" />
             <geometry>
-                <mesh filename="package://sobot/description/meshes/sobot_wheel.dae" scale="1 1 1"/> <!-- Colocar o arquivo STL-->
+                <mesh filename="package://sobot_drive/meshes/sobot_wheel.dae" scale="1 1 1"/> <!-- Colocar o arquivo STL-->
             </geometry>
         </visual>

Commit message: Alterações api

File: install/sobot_drive/share/sobot_drive/ros2_control/diffbot.ros2_control.xacro (robot description, xacro)
@@ -1,33 +1 @@
-<?xml version="1.0"?>
-<robot xmlns:xacro="http://www.ros.org/wiki/xacro">
-  <xacro:macro name="diffbot_ros2_control" params="name prefix use_mock_hardware">
-    <ros2_control name="${name}" type="system">
-      <xacro:unless value="${use_mock_hardware}">
-        <hardware>
-          <plugin>sobot_drive/SobotDriveHardware</plugin>
-          <param name="example_param_hw_start_duration_sec">0</param>
-          <param name="example_param_hw_stop_duration_sec">3.0</param>
-          <param name="device">/dev/ttyACM0</param>
-          <param name="baud_rate">57600</param>
-          <param name="timeout_ms">1000</param>
-        </hardware>
-      </xacro:unless>
-      <xacro:if value="${use_mock_hardware}">
-        <hardware>
-          <plugin>mock_components/GenericSystem</plugin>
-          <param name="calculate_dynamics">true</param>
-        </hardware>
-      </xacro:if>
-      <joint name="${prefix}left_wheel_joint">
-        <command_interface name="velocity"/>
-        <state_interface name="position"/>
-        <state_interface name="velocity"/>
-      </joint>
-      <joint name="${prefix}right_wheel_joint">
-        <command_interface name="velocity"/>
-        <state_interface name="position"/>
-        <state_interface name="velocity"/>
-      </joint>
-    </ros2_control>
-  </xacro:macro>
-</robot>
+/dev_ws/src/sobot_drive/description/ros2_control/diffbot.ros2_control.xacro

File: install/sobot_drive/share/sobot_drive/urdf/diffbot.urdf.xacro (robot description, xacro)
@@ -1,11 +1 @@
-<?xml version="1.0"?>
-<!-- Basic differential drive mobile base -->
-<robot xmlns:xacro="http://www.ros.org/wiki/xacro" name="diffdrive_robot">
-  <xacro:arg name="prefix" default="" />
-  <xacro:arg name="use_mock_hardware" default="false" />
-  <xacro:include filename="robot_core.xacro" />
-  <!-- Import diffbot ros2_control description -->
-  <xacro:include filename="$(find sobot_drive)/ros2_control/diffbot.ros2_control.xacro" />
-  <xacro:diffbot_ros2_control
-    name="DiffBot" prefix="$(arg prefix)" use_mock_hardware="$(arg use_mock_hardware)"/>
-</robot>
+/dev_ws/src/sobot_drive/description/urdf/diffbot.urdf.xacro

File: src/sobot_drive/description/ros2_control/diffbot.ros2_control.xacro (robot description, xacro)
@@ -11,4 +11,7 @@
           <param name="baud_rate">57600</param>
           <param name="timeout_ms">1000</param>
+          <param name="update_rate">10</param>
+          <param name="wheel_separation">0.264</param>
+          <param name="wheel_radius">0.05</param>
         </hardware>
       </xacro:unless>
