Commit message: Att nav2

File: src/sobot_gazebo/description/urdf/robot.urdf.xacro (robot description, xacro)
@@ -4,3 +4,4 @@
     <!-- <xacro:include filename="gazebo_control.xacro" /> -->
     <xacro:include filename="ros2_control_sim.xacro" />
+    <xacro:include filename="lidar.xacro" />
 </robot>

File: src/sobot_gazebo/description/urdf/robot_core.xacro (robot description, xacro)
@@ -22,4 +22,12 @@
     <!-- BASE LINK -->
     <link name="base_link">
+    </link>
+    <!-- BASE_FOOTPRINT LINK-->
+    <joint name="base_footprint_joint" type="fixed">
+        <parent link="base_link"/>
+        <child link="base_footprint"/>
+        <origin xyz="0 0 0" rpy="0 0 0"/>
+    </joint>
+    <link name="base_footprint">
     </link>
     <!-- CHASSIS LINK -->
